Commit message: [Phy] Refined Physics and Made Final Internship Prototype

File: assets/drone.urdf (robot description, URDF)
Before this commit: robot drone, 13 links, 12 joints
Links:
- link arm_bl: mass 0.01 -> 0.04; geometry collision box size=0.184 0.02 0.02; visual box size=0.184 0.02 0.02
- link arm_br: mass 0.01 -> 0.04; geometry collision box size=0.184 0.02 0.02; visual box size=0.184 0.02 0.02
- link arm_fl: mass 0.01 -> 0.04; geometry collision box size=0.184 0.02 0.02; visual box size=0.184 0.02 0.02
- link arm_fr: mass 0.01 -> 0.04; geometry collision box size=0.184 0.02 0.02; visual box size=0.184 0.02 0.02
- link base_link: mass 0.18 -> 0.72; geometry collision cylinder length=0.04 radius=0.14; visual cylinder length=0.04 radius=0.14
- link motor_bl: mass 0.005 -> 0.02; geometry collision cylinder length=0.04 radius=0.03; visual cylinder length=0.04 radius=0.03
- link motor_br: mass 0.005 -> 0.02; geometry collision cylinder length=0.04 radius=0.03; visual cylinder length=0.04 radius=0.03
- link motor_fl: mass 0.005 -> 0.02; geometry collision cylinder length=0.04 radius=0.03; visual cylinder length=0.04 radius=0.03
- link motor_fr: mass 0.005 -> 0.02; geometry collision cylinder length=0.04 radius=0.03; visual cylinder length=0.04 radius=0.03
- link prop_bl: mass 0.005 -> 0.02; geometry collision cylinder length=0.006 radius=0.12; visual cylinder length=0.006 radius=0.12
- link prop_br: mass 0.005 -> 0.02; geometry collision cylinder length=0.006 radius=0.12; visual cylinder length=0.006 radius=0.12
- link prop_fl: mass 0.005 -> 0.02; geometry collision cylinder length=0.006 radius=0.12; visual cylinder length=0.006 radius=0.12
- link prop_fr: mass 0.005 -> 0.02; geometry collision cylinder length=0.006 radius=0.12; visual cylinder length=0.006 radius=0.12
Joints:
- joint joint_arm_bl: origin xyz=-0.0381 0.0381 0 rpy=0 0 2.3562 -> xyz=-0.0762 0.0762 0 rpy=0 0 2.3562
- joint joint_arm_br: origin xyz=-0.0381 -0.0381 0 rpy=0 0 -2.3562 -> xyz=-0.0762 -0.0762 0 rpy=0 0 -2.3562
- joint joint_arm_fl: origin xyz=0.0381 0.0381 0 rpy=0 0 0.7854 -> xyz=0.0762 0.0762 0 rpy=0 0 0.7854
- joint joint_arm_fr: origin xyz=0.0381 -0.0381 0 rpy=0 0 -0.7854 -> xyz=0.0762 -0.0762 0 rpy=0 0 -0.7854
- joint joint_motor_bl: origin xyz=-0.0919 0.0919 0 rpy=0 0 0 -> xyz=-0.1838 0.1838 0 rpy=0 0 0
- joint joint_motor_br: origin xyz=-0.0919 -0.0919 0 rpy=0 0 0 -> xyz=-0.1838 -0.1838 0 rpy=0 0 0
- joint joint_motor_fl: origin xyz=0.0919 0.0919 0 rpy=0 0 0 -> xyz=0.1838 0.1838 0 rpy=0 0 0
- joint joint_motor_fr: origin xyz=0.0919 -0.0919 0 rpy=0 0 0 -> xyz=0.1838 -0.1838 0 rpy=0 0 0
- joint joint_prop_bl: origin xyz=0 0 0.01 rpy=0 0 0 -> xyz=0 0 0.02 rpy=0 0 0
- joint joint_prop_br: origin xyz=0 0 0.01 rpy=0 0 0 -> xyz=0 0 0.02 rpy=0 0 0
- joint joint_prop_fl: origin xyz=0 0 0.01 rpy=0 0 0 -> xyz=0 0 0.02 rpy=0 0 0
- joint joint_prop_fr: origin xyz=0 0 0.01 rpy=0 0 0 -> xyz=0 0 0.02 rpy=0 0 0
